Commit message: Add stand-mounted RealSense D415 to simulation
Apply materials to the stand model
Realsense gazebo xacro lifted from Astro (Fetch) simulation

File: aurmr_gazebo/robots/tahoma.gazebo.xacro (robot description, xacro)
@@ -2,4 +2,5 @@
   <xacro:include filename="$(find tahoma_description)/robots/tahoma.xacro"/>
   <xacro:include filename="$(find aurmr_gazebo)/urdf/robotiq_2f_85_gazebo_macro.xacro" />
+  <xacro:include filename="$(find aurmr_gazebo)/urdf/d415.gazebo.xacro"/>
   <xacro:robotiq_2f_85_gazebo prefix="gripper_" />
   <!-- Configure self collision properties per link -->
@@ -29,9 +30,80 @@
     </plugin>
   </gazebo>
+  <gazebo reference="stand">
+      <material>AURMR/BlueAluminum</material>
+  </gazebo>
+  <gazebo reference="stand_brace">
+      <material>AURMR/BlueAluminum</material>
+  </gazebo>
+  <gazebo reference="stand_upright">
+      <material>AURMR/BlueAluminum</material>
+  </gazebo>
+  <gazebo reference="robot_beam">
+    <material>AURMR/BlueAluminum</material>
+  </gazebo>
+    <gazebo reference="control_box_mount">
+    <material>AURMR/BlueAluminum</material>
+  </gazebo>
+      <gazebo reference="front_left_caster">
+    <material>Gazebo/Gray</material>
+  </gazebo>
+        <gazebo reference="front_right_caster">
+    <material>Gazebo/Gray</material>
+  </gazebo>
+        <gazebo reference="back_left_caster">
+    <material>Gazebo/Gray</material>
+  </gazebo>
+        <gazebo reference="back_right_caster">
+    <material>Gazebo/Gray</material>
+  </gazebo>
+  <xacro:if value="${'$(arg realsense)' == 'false' }">
+    <gazebo reference="mid_camera_depth_frame">
+      <sensor type="camera" name="depth_camera">
+        <update_rate>6.0</update_rate>
+        <camera name="depth">
+          <horizontal_fov>1.047198</horizontal_fov>
+          <image>
+            <width>640</width>
+            <height>480</height>
+            <format>R8G8B8</format>
+          </image>
+          <clip>
+            <near>0.02</near>
+            <far>100</far>
+          </clip>
+          <noise>
+            <type>gaussian</type>
+            <!-- Noise is sampled independently per pixel on each frame.
+                 That pixel's noise value is added to each of its color
+                 channels, which at that point lie in the range [0,1]. -->
+            <mean>0.0</mean>
+            <stddev>0.007</stddev>
+          </noise>
+        </camera>
+        <plugin name="camera_controller" filename="libgazebo_ros_camera.so">
+          <alwaysOn>false</alwaysOn>
+          <updateRate>0.0</updateRate>
+          <cameraName>camera</cameraName>
+          <imageTopicName>color/image_raw</imageTopicName>
+          <cameraInfoTopicName>color/camera_info</cameraInfoTopicName>
+          <frameName>camera_depth_optical_frame</frameName>
+          <hackBaseline>0.07</hackBaseline>
+          <distortionK1>0.0</distortionK1>
+          <distortionK2>0.0</distortionK2>
+          <distortionK3>0.0</distortionK3>
+          <distortionT1>0.0</distortionT1>
+          <distortionT2>0.0</distortionT2>
+        </plugin>
+      </sensor>
+    </gazebo>
+  </xacro:if>
+  <xacro:if value="${'$(arg realsense)' == 'true' }">
+        <xacro:sensor_d415_gazebo name="mid_camera"/>
+  </xacro:if>
   <link name="world"/>
   <joint name="world_joint" type="fixed">
     <parent link="world"/>
     <child link="base_link"/>
-    <origin xyz="0 0 .5" rpy="0 0 0"/>
+    <origin xyz="0 0 0" rpy="0 0 0"/>
   </joint>
 </robot>

Commit message: Tweak Tahoma model
Adjust aluminum material to be darker, closer match
Add materials to some new links
Remove fixed ground joint which we seem fine without now that the stand model has reasonable inertial markup
Add l515 plugin hookup, but disable until I can make it work

File: aurmr_gazebo/robots/tahoma.gazebo.xacro (robot description, xacro)
@@ -1,7 +1,9 @@
 <robot xmlns:xacro="http://www.ros.org/wiki/xacro" name="tahoma">
   <xacro:include filename="$(find tahoma_description)/robots/tahoma.xacro"/>
-  <xacro:include filename="$(find aurmr_gazebo)/urdf/robotiq_2f_85_gazebo_macro.xacro" />
+  <xacro:include filename="$(find aurmr_gazebo)/urdf/robotiq_2f_85_gazebo_macro.xacro"/>
+  <xacro:include filename="$(find aurmr_gazebo)/urdf/l515.gazebo.xacro"/>
   <xacro:include filename="$(find aurmr_gazebo)/urdf/d415.gazebo.xacro"/>
-  <xacro:robotiq_2f_85_gazebo prefix="gripper_" />
+  <xacro:robotiq_2f_85_gazebo prefix="gripper_"/>
+  <xacro:arg name="realsense" default="true" />
   <!-- Configure self collision properties per link -->
   <gazebo reference="arm_shoulder_link">
@@ -31,29 +33,47 @@
   </gazebo>
   <gazebo reference="stand">
-      <material>AURMR/BlueAluminum</material>
+    <material>AURMR/BlueAluminum</material>
   </gazebo>
   <gazebo reference="stand_brace">
-      <material>AURMR/BlueAluminum</material>
+    <material>AURMR/BlueAluminum</material>
   </gazebo>
   <gazebo reference="stand_upright">
-      <material>AURMR/BlueAluminum</material>
-  </gazebo>
-  <gazebo reference="robot_beam">
     <material>AURMR/BlueAluminum</material>
   </gazebo>
-    <gazebo reference="control_box_mount">
+  <gazebo reference="cantilever">
     <material>AURMR/BlueAluminum</material>
   </gazebo>
-      <gazebo reference="front_left_caster">
+  <gazebo reference="control_box_mount">
+    <material>AURMR/BlueAluminum</material>
+  </gazebo>
+  <gazebo reference="control_box">
     <material>Gazebo/Gray</material>
   </gazebo>
-        <gazebo reference="front_right_caster">
+  <gazebo reference="robot_plate">
+    <material>AURMR/BlueAluminum</material>
+  </gazebo>
+  <gazebo reference="front_left_caster">
     <material>Gazebo/Gray</material>
   </gazebo>
-        <gazebo reference="back_left_caster">
+  <gazebo reference="front_right_caster">
     <material>Gazebo/Gray</material>
   </gazebo>
-        <gazebo reference="back_right_caster">
+  <gazebo reference="back_left_caster">
     <material>Gazebo/Gray</material>
+  </gazebo>
+  <gazebo reference="back_right_caster">
+    <material>Gazebo/Gray</material>
+  </gazebo>
+  <gazebo reference="left_light_panel">
+    <material>Gazebo/Gray</material>
+  </gazebo>
+  <gazebo reference="right_light_panel">
+    <material>Gazebo/Gray</material>
+  </gazebo>
+  <gazebo reference="left_light_panel_emitter">
+    <material>Gazebo/WhiteGlow</material>
+  </gazebo>
+  <gazebo reference="right_light_panel_emitter">
+    <material>Gazebo/WhiteGlow</material>
   </gazebo>
   <xacro:if value="${'$(arg realsense)' == 'false' }">
@@ -99,11 +119,6 @@
   </xacro:if>
   <xacro:if value="${'$(arg realsense)' == 'true' }">
-        <xacro:sensor_d415_gazebo name="mid_camera"/>
+    <!--xacro:sensor_l515_gazebo name="stand_camera"/-->
+    <xacro:sensor_d415_gazebo name="stand_camera"/>
   </xacro:if>
-  <link name="world"/>
-  <joint name="world_joint" type="fixed">
-    <parent link="world"/>
-    <child link="base_link"/>
-    <origin xyz="0 0 0" rpy="0 0 0"/>
-  </joint>
 </robot>

File: aurmr_gazebo/urdf/d415.gazebo.xacro (robot description, xacro)
@@ -6,5 +6,5 @@
 aluminum peripherial evaluation case.
 -->
-<robot name="sensor-d415-gazebo" xmlns:xacro="http://ros.org/wiki/xacro">
+<robot  xmlns:xacro="http://ros.org/wiki/xacro">
     <xacro:macro name="sensor_d415_gazebo" params="name:=camera ">
         <xacro:property name="M_PI" value="3.1415926535897931"/>

Commit message: Paste in l515 gazebo plugin
Functions correctly with the L515 URDF, but not checked against the real sensor
It seems like PAL's realsense gazebo plugin (which this one is a fork of) hardcodes some use of the two infrared streams for the stereo depth cameras. This fork seems to just cut those out

File: aurmr_gazebo/robots/tahoma.gazebo.xacro (robot description, xacro)
@@ -119,6 +119,5 @@
   </xacro:if>
   <xacro:if value="${'$(arg realsense)' == 'true' }">
-    <!--xacro:sensor_l515_gazebo name="stand_camera"/-->
-    <xacro:sensor_d415_gazebo name="stand_camera"/>
+    <xacro:sensor_l515_gazebo name="stand_camera"/>
   </xacro:if>
 </robot>

File: aurmr_gazebo/urdf/l515.gazebo.xacro (robot description, xacro)
@@ -6,5 +6,5 @@
 -->
 <robot xmlns:xacro="http://ros.org/wiki/xacro">
-  <xacro:macro name="sensor_l515_gazebo" params="name  publish_pointcloud:=true" >
+  <xacro:macro name="sensor_l515_gazebo" params="name  publish_pointcloud:=false" >
     <!-- Load parameters to model's main link-->
     <xacro:property name="deg_to_rad" value="0.01745329251994329577" />
@@ -28,5 +28,5 @@
           </image>
           <clip>
-            <near>0.1</near>
+            <near>0.01</near>
             <far>100</far>
           </clip>
@@ -39,5 +39,5 @@
         <always_on>1</always_on>
         <update_rate>30</update_rate>
-        <visualize>1</visualize>
+        <visualize>0</visualize>
       </sensor>
       <sensor name="${name}ired" type="camera">
@@ -50,6 +50,6 @@
           </image>
           <clip>
-            <near>0.1</near>
-            <far>100</far>
+            <near>0.25</near>
+            <far>6.5</far>
           </clip>
           <noise>
@@ -60,5 +60,5 @@
         </camera>
         <always_on>1</always_on>
-        <update_rate>90</update_rate>
+        <update_rate>30</update_rate>
         <visualize>0</visualize>
       </sensor>
@@ -71,6 +71,6 @@
           </image>
           <clip>
-            <near>0.1</near>
-            <far>100</far>
+            <near>0.25</near>
+            <far>6.5</far>
           </clip>
           <noise>
@@ -81,10 +81,10 @@
         </camera>
         <always_on>1</always_on>
-        <update_rate>90</update_rate>
+        <update_rate>30</update_rate>
         <visualize>0</visualize>
       </sensor>
     </gazebo>
     <gazebo>
-      <plugin name="${name}" filename="librealsense_gazebo_plugin.so">
+      <plugin name="${name}" filename="librealsense_l515_gazebo_plugin.so">
         <prefix>${name}</prefix>
         <depthUpdateRate>30.0</depthUpdateRate>
@@ -101,5 +101,5 @@
         <infraredOpticalframeName>${name}_infra_optical_frame</infraredOpticalframeName>
         <rangeMinDepth>0.2</rangeMinDepth>
-        <rangeMaxDepth>10.0</rangeMaxDepth>
+        <rangeMaxDepth>6.5</rangeMaxDepth>
         <pointCloud>${publish_pointcloud}</pointCloud>
         <pointCloudTopicName>depth/color/points</pointCloudTopicName>

Commit message: Tweak colors, materials
Add noisy fabric texture to pod fabric
Tone down strong ceiling light
Add light sources to world that mimic light panels so the shading on the bins looks more appropriate

File: aurmr_gazebo/robots/tahoma.gazebo.xacro (robot description, xacro)
@@ -32,4 +32,7 @@
     </plugin>
   </gazebo>
+    <gazebo reference="coupling">
+        <material>Gazebo/Black</material>
+    </gazebo>
   <gazebo reference="stand">
     <material>AURMR/BlueAluminum</material>
@@ -39,4 +42,7 @@
   </gazebo>
   <gazebo reference="stand_upright">
+    <material>AURMR/BlueAluminum</material>
+  </gazebo>
+    <gazebo reference="camera_beam_lower">
     <material>AURMR/BlueAluminum</material>
   </gazebo>

Commit message: Use new Tahoma xacro macro
Removes the need for the launch file to pass an argument. We know that the simulation will always have to use these fake extrinsics, so configuring this in the tahoma.gazebo.xacro ensures this

File: aurmr_gazebo/robots/tahoma.gazebo.xacro (robot description, xacro)
@@ -1,8 +1,9 @@
 <robot xmlns:xacro="http://www.ros.org/wiki/xacro" name="tahoma">
-  <xacro:include filename="$(find tahoma_description)/robots/tahoma.xacro"/>
+  <xacro:arg name="realsense" default="true" />
+  <xacro:include filename="$(find tahoma_description)/urdf/tahoma.xacro"/>
   <xacro:include filename="$(find aurmr_gazebo)/urdf/robotiq_2f_85_gazebo_macro.xacro"/>
   <xacro:include filename="$(find aurmr_gazebo)/urdf/l515.gazebo.xacro"/>
+  <xacro:tahoma use_nominal_camera_extrinsics="true"/>
   <xacro:robotiq_2f_85_gazebo prefix="gripper_"/>
-  <xacro:arg name="realsense" default="true" />
   <!-- Configure self collision properties per link -->
   <gazebo reference="arm_shoulder_link">
@@ -31,7 +32,7 @@
     </plugin>
   </gazebo>
-    <gazebo reference="coupling">
-        <material>Gazebo/Black</material>
-    </gazebo>
+  <gazebo reference="coupling">
+      <material>Gazebo/Black</material>
+  </gazebo>
   <gazebo reference="stand">
     <material>AURMR/BlueAluminum</material>
