Commit message: fc.launch file includes new parameters (rpy, binRandPoseN, etc). common.xml file doesn't spawn pod when fc.launch file is run (i.e. spawning pod only once), but instead initializes node 'analyze_workspace' where pod is programmaticaly spawned over range of xy. spawn_tahoma.xml doesn't set home pose of the robot as the simulation in Gazebo starts immediately (previously it was paused to adjust robot to home pose). pod.gazebo.xacro is renamed to pod1.gazebo.xacro (pod with 13x4 small bins). pod2.gazebo.xacro is created for the pod with 8x3 large bins

File: aurmr_gazebo/robots/pod1.gazebo.xacro (robot description, xacro)
@@ -1,9 +1,10 @@
+<?xml version="1.0"?>
 <robot xmlns:xacro="http://www.ros.org/wiki/xacro" name="pod">
-  <xacro:arg name="id" default="" />
+  <xacro:arg name="id" default="1" />
   <xacro:arg name="fixed" default="true" />
   <xacro:include filename="$(find tahoma_description)/robots/pod$(arg id).xacro"/>
   <xacro:if value="$(arg fixed)">
     <link name="world"/>
-    <joint name="fixed" type="fixed">
+    <joint name="fixed" type="floating">
         <parent link="world"/>
         <child link="pod_base_link"/>

File: aurmr_gazebo/robots/tahoma.gazebo.xacro (robot description, xacro)
@@ -28,11 +28,17 @@
     <selfCollide>true</selfCollide>
   </gazebo>
+  <gazebo reference="arm_wrist_2_link">
+    <selfCollide>true</selfCollide>
+  </gazebo>
   <gazebo reference="arm_wrist_3_link">
     <selfCollide>true</selfCollide>
   </gazebo>
-  <gazebo reference="arm_wrist_2_link">
+  <gazebo reference="gripper_base_link">
     <selfCollide>true</selfCollide>
   </gazebo>
-  <gazebo reference="arm_ee_link">
+  <gazebo reference="epick_end_effector">
+    <selfCollide>true</selfCollide>
+  </gazebo>
+  <gazebo reference="connector_cover">
     <selfCollide>true</selfCollide>
   </gazebo>
@@ -42,4 +48,7 @@
   </gazebo>
   <gazebo reference="coupling">
+      <material>Gazebo/Black</material>
+  </gazebo>
+  <gazebo reference="connector_cover">
       <material>Gazebo/Black</material>
   </gazebo>
