Commit message: Update pod model wrapper
Wrap flap link

File: aurmr_gazebo/robots/pod.gazebo.xacro (robot description, xacro)
@@ -6,5 +6,5 @@
   <xacro:macro name="color_pod_fabric" params="prefix">
     <xacro:arg name="prefix" default=""/>
-    <xacro:property name="front_recipe" value="${[0,0,0,0,0,0,0,0,0,0,0,0,0]}"/>
+    <xacro:property name="recipe_a" value="${[0,0,0,0,0,0,0,0,0,0,0,0,0]}"/>
     <xacro:property name="alphabet" value="abcdefghijklmnopqrstuvwxyz"/>
     <xacro:macro name="shifted_box" params="name">
@@ -20,4 +20,5 @@
       <xacro:shifted_box name="${bin_name}_top" />
       <xacro:shifted_box name="${bin_name}_back" />
+      <xacro:shifted_box name="${bin_name}_flap" />
     </xacro:macro>
     <xacro:macro name="bin_row" params="prefix:=^ id parent sections  i:=0">
@@ -41,5 +42,5 @@
       </xacro:if>
     </xacro:macro>
-    <xacro:shelf_stack prefix="pod_" parent="${prefix}fabric_base" recipe="${front_recipe}"/>
+    <xacro:shelf_stack prefix="pod_" parent="${prefix}fabric_base" recipe="${recipe_a}"/>
   </xacro:macro>
   <xacro:color_pod_fabric prefix="pod_" />

Commit message: Make pod and robot fixed to scene by default
The robot still jitters, but now the pod can handle getting objects spawned inside it

File: aurmr_gazebo/robots/pod.gazebo.xacro (robot description, xacro)
@@ -1,5 +1,13 @@
-<robot xmlns:xacro="http://www.ros.org/wiki/xacro" name="pod" params="id">
+<robot xmlns:xacro="http://www.ros.org/wiki/xacro" name="pod">
   <xacro:arg name="id" default="" />
+  <xacro:arg name="fixed" default="true" />
   <xacro:include filename="$(find tahoma_description)/robots/pod$(arg id).xacro"/>
+  <xacro:if value="$(arg fixed)">
+    <link name="world"/>
+    <joint name="fixed" type="fixed">
+        <parent link="world"/>
+        <child link="pod_base_link"/>
+    </joint>
+  </xacro:if>
   <gazebo reference="pod_base_link">
     <material>Gazebo/Gray</material>

File: aurmr_gazebo/robots/tahoma.gazebo.xacro (robot description, xacro)
@@ -1,7 +1,15 @@
-<robot xmlns:xacro="http://www.ros.org/wiki/xacro" name="tahoma">
+<robot xmlns:xacro="http://www.ros.org/wiki/xacro" name="tahoma" >
+  <xacro:arg name="fixed" default="true" />
   <xacro:arg name="realsense" default="true" />
   <xacro:include filename="$(find tahoma_description)/urdf/tahoma.xacro"/>
   <xacro:include filename="$(find aurmr_gazebo)/urdf/robotiq_2f_85_gazebo_macro.xacro"/>
   <xacro:include filename="$(find aurmr_gazebo)/urdf/l515.gazebo.xacro"/>
+  <xacro:if value="$(arg fixed)">
+    <link name="world"/>
+    <joint name="fixed" type="fixed">
+        <parent link="world"/>
+        <child link="base_link"/>
+    </joint>
+  </xacro:if>
   <xacro:tahoma use_nominal_camera_extrinsics="true" gripper_transmission_hw_interface="hardware_interface/PositionJointInterface"/>
   <xacro:robotiq_2f_85_gazebo prefix="gripper_"/>

Commit message: IMPL: launch/xml files are adjusted for single xacro files of pods

File: aurmr_gazebo/robots/pod.gazebo.xacro (robot description, xacro)
@@ -1,8 +1,9 @@
 <?xml version="1.0"?>
 <robot xmlns:xacro="http://www.ros.org/wiki/xacro" name="pod">
-  <xacro:arg name="id" default="1A" />
+  <xacro:arg name="id" default="1B" />
+  <xacro:arg name="include_flaps" default="true" />
   <xacro:arg name="fixed" default="true" />
   <xacro:include filename="$(find tahoma_description)/robots/pod.xacro"/>
-  <xacro:pod_recipe id="$(arg id)"/>
+  <xacro:pod_recipe pod_id="$(arg id)" include_flaps="$(arg include_flaps)"/>
   <!-- Scripts below are just to paint the pod (bins & ) in Gazebo scene -->
   <xacro:if value="$(arg fixed)">
@@ -57,7 +58,8 @@
       </gazebo>
     </xacro:macro>
-    <xacro:macro name="bin" params="prefix colrow_id rightmost:=false top_shelf:=false">
+    <xacro:macro name="bin" params="prefix colrow_id rightmost:=false">
       <xacro:property name="bin_name" value="${prefix}bin_${colrow_id}"/>
       <xacro:shifted_box name="${bin_name}_bottom"/>
+      <xacro:shifted_box name="${bin_name}_top"/>
       <xacro:shifted_box name="${bin_name}_left"/>
       <xacro:shifted_box name="${bin_name}_back"/>
@@ -66,9 +68,6 @@
         <xacro:shifted_box name="${bin_name}_right"/>
       </xacro:if>
-      <xacro:if value="${top_shelf}">
-        <xacro:shifted_box name="${bin_name}_top"/>
-      </xacro:if>
     </xacro:macro>
-    <xacro:macro name="bin_row" params="prefix row_id bin_row_base sections i:=0 top_shelf:=false">
+    <xacro:macro name="bin_row" params="prefix row_id bin_row_base sections i:=0">
       <xacro:property name="bin_name" value="${prefix}bin_${i+1}${row_id}"/>
       <xacro:if value="${sections == 1}">
@@ -78,41 +77,37 @@
         <xacro:property name="rightmost" value="false"/>
       </xacro:unless>
-      <xacro:bin prefix="${prefix}" colrow_id="${i+1}${row_id}" rightmost="${rightmost}" top_shelf="${top_shelf}"/>
+      <xacro:bin prefix="${prefix}" colrow_id="${i+1}${row_id}" rightmost="${rightmost}"/>
       <xacro:if value="${sections > 1}"><!-- recurse for the remaining bins -->
-        <xacro:bin_row prefix="${prefix}" row_id="${row_id}" bin_row_base="${bin_row_base}" sections="${sections-1}" i="${i+1}" top_shelf="${top_shelf}"/>
+        <xacro:bin_row prefix="${prefix}" row_id="${row_id}" bin_row_base="${bin_row_base}" sections="${sections-1}" i="${i+1}"/>
       </xacro:if>
     </xacro:macro>
-    <xacro:macro name="shelf" params="prefix row_id sections:=4 top_shelf:=false">
+    <xacro:macro name="shelf" params="prefix row_id sections:=4">
       <xacro:property name="shelf_name" value="${prefix}shelf_${row_id}"/>
       <xacro:if value="${X_OFFSET != 0}"><!-- left margin, relates to B & D faces of pods -->
         <xacro:shifted_box name="${shelf_name}_left_margin"/>
       </xacro:if>
-      <xacro:bin_row prefix="${prefix}" row_id="${row_id}" bin_row_base="${shelf_name}" sections="${sections}" top_shelf="${top_shelf}"/>
+      <xacro:bin_row prefix="${prefix}" row_id="${row_id}" bin_row_base="${shelf_name}" sections="${sections}"/>
       <xacro:if value="${X_OFFSET != 0}"><!-- left margin, relates to B & D faces of pods -->
         <xacro:shifted_box name="${shelf_name}_right_margin"/>
       </xacro:if>
     </xacro:macro>
-    <xacro:macro name="shelf_stack" params="prefix shelf_stack_base shelf_heights i:=0">
+    <xacro:macro name="shelf_stack" params="prefix shelf_heights i:=0">
       <xacro:property name="shelf_name" value="${prefix}shelf_${alphabet[i]}"/>
       <xacro:if value="${FACE_ID == 'B' or FACE_ID == 'D'}">
-        <xacro:if value="${POD_ID == '1' and i == 0}">
+        <xacro:if value="${POD_ID == 1 and i == 0}">
           <xacro:property name="NUM_COLUMNS" value="1"/>
         </xacro:if>
-        <xacro:unless value="${POD_ID == '1' and i == 0}">
-          <xacro:property name="NUM_COLUMNS" value="2"/>
+        <xacro:unless value="${POD_ID == 1 and i == 0}">
+          <xacro:if value="${POD_ID == 1}">
+            <xacro:property name="NUM_COLUMNS" value="2"/>
+          </xacro:if>
         </xacro:unless>
       </xacro:if>
-      <xacro:if value="${len(shelf_heights) == 1}">
-        <xacro:property name="top_shelf" value="true"/>
-      </xacro:if>
-      <xacro:unless value="${len(shelf_heights) == 1}">
-        <xacro:property name="top_shelf" value="false"/>
-      </xacro:unless>
-      <xacro:shelf prefix="${prefix}" row_id="${alphabet[i]}" sections="${NUM_COLUMNS}" top_shelf="${top_shelf}"/>
+      <xacro:shelf prefix="${prefix}" row_id="${alphabet[i]}" sections="${NUM_COLUMNS}"/>
       <xacro:if value="${len(shelf_heights) > 1}"><!-- recurse for the remaining shelves -->
-        <xacro:shelf_stack prefix="${prefix}" shelf_stack_base="${shelf_stack_base}" shelf_heights="${shelf_heights[1:]}" i="${i+1}"/>
+        <xacro:shelf_stack prefix="${prefix}" shelf_heights="${shelf_heights[1:]}" i="${i+1}"/>
       </xacro:if>
     </xacro:macro>
-    <xacro:shelf_stack prefix="pod_" shelf_stack_base="${prefix}fabric_base" shelf_heights="${BIN_HEIGHTS}"/>
+    <xacro:shelf_stack prefix="pod_" shelf_heights="${BIN_HEIGHTS}"/>
   </xacro:macro>
   <xacro:color_pod_fabric prefix="pod_"/>

File: aurmr_gazebo/robots/tahoma.gazebo.xacro (robot description, xacro)
@@ -2,8 +2,8 @@
 <robot xmlns:xacro="http://www.ros.org/wiki/xacro" name="tahoma" >
   <xacro:arg name="fixed" default="true" />
-  <xacro:arg name="realsense" default="true" />
+  <!-- <xacro:arg name="realsense" default="true" /> -->
   <xacro:include filename="$(find tahoma_description)/urdf/tahoma.xacro"/>
   <xacro:include filename="$(find aurmr_gazebo)/urdf/robotiq_epick.gazebo.xacro"/>
-  <xacro:include filename="$(find aurmr_gazebo)/urdf/l515.gazebo.xacro"/>
+  <!-- <xacro:include filename="$(find aurmr_gazebo)/urdf/l515.gazebo.xacro"/> -->
   <xacro:if value="$(arg fixed)">
     <link name="world"/>
@@ -13,5 +13,5 @@
     </joint>
   </xacro:if>
-  <xacro:tahoma use_nominal_camera_extrinsics="true" gripper_transmission_hw_interface="hardware_interface/PositionJointInterface"/>
+  <xacro:tahoma use_nominal_camera_extrinsics="true"/>
   <xacro:epick_hand_gazebo robot_name="tahoma"/>
   <!-- Configure self collision properties per link -->
@@ -43,4 +43,5 @@
     <selfCollide>true</selfCollide>
   </gazebo>
+  <!-- gazebo_ros_control -->
   <gazebo>
     <plugin name="ros_control" filename="libgazebo_ros_control.so">
@@ -101,5 +102,6 @@
     <material>Gazebo/WhiteGlow</material>
   </gazebo>
-  <xacro:if value="${'$(arg realsense)' == 'false' }">
+</robot>
+  <!-- <xacro:if value="${'$(arg realsense)' == 'false' }">
     <gazebo reference="mid_camera_depth_frame">
       <sensor type="camera" name="depth_camera">
@@ -117,9 +119,9 @@
           </clip>
           <noise>
-            <type>gaussian</type>
+            <type>gaussian</type> -->
             <!-- Noise is sampled independently per pixel on each frame.
                  That pixel's noise value is added to each of its color
                  channels, which at that point lie in the range [0,1]. -->
-            <mean>0.0</mean>
+            <!-- <mean>0.0</mean>
             <stddev>0.007</stddev>
           </noise>
@@ -141,8 +143,7 @@
       </sensor>
     </gazebo>
-  </xacro:if>
+  </xacro:if> -->
   <!--<xacro:if value="${'$(arg realsense)' == 'true' }">
     <xacro:sensor_l515_gazebo name="camera_lower_left"/>
     <xacro:sensor_l515_gazebo name="camera_lower_right"/>
   </xacro:if> -->
-</robot>
