Commit message: Tweak l515 xacro
Use radians/1 helper

File: aurmr_gazebo/urdf/l515.gazebo.xacro (robot description, xacro)
@@ -8,5 +8,4 @@
   <xacro:macro name="sensor_l515_gazebo" params="name  publish_pointcloud:=false" >
     <!-- Load parameters to model's main link-->
-    <xacro:property name="deg_to_rad" value="0.01745329251994329577" />
     <gazebo reference="${name}_link">
       <self_collide>0</self_collide>
@@ -21,5 +20,5 @@
       <sensor name="${name}color" type="camera">
         <camera name="${name}">
-          <horizontal_fov>${71.01*deg_to_rad}</horizontal_fov>
+          <horizontal_fov>${radians(71.01)}</horizontal_fov>
           <image>
             <width>1920</width>
@@ -43,5 +42,5 @@
       <sensor name="${name}ired" type="camera">
         <camera name="${name}">
-          <horizontal_fov>${70*deg_to_rad}</horizontal_fov>
+          <horizontal_fov>${radians(70)}</horizontal_fov>
           <image>
             <width>1024</width>
@@ -65,5 +64,5 @@
       <sensor name="${name}depth" type="depth">
         <camera name="${name}">
-          <horizontal_fov>${70*deg_to_rad}</horizontal_fov>
+          <horizontal_fov>${radians(70)}</horizontal_fov>
           <image>
             <width>1024</width>
